File: kicad/Esp32LoraBoard/Esp32LoraBoard.kicad_pcb (KiCad board)
At the start: 2 copper layers, 71.8 x 64.1 mm, 13 parts, among them J1 USB_B_Micro, J2 Power-Selector, J3 Testpoints, U1 LM3940IMP-3.3, U2 ESP32-WROOM-32, U3 RFM95W-868S2

Commit message: .
Parts:
- added C5: 1n, Capacitor_SMD:C_1206_3216Metric_Pad1.42x1.75mm_HandSolder, F.Cu at (128.5, 64.0)
- added C6: 1n, Capacitor_SMD:C_1206_3216Metric_Pad1.42x1.75mm_HandSolder, F.Cu at (157.0, 85.6)
- added C7: 100n, Capacitor_SMD:C_1206_3216Metric_Pad1.42x1.75mm_HandSolder, F.Cu at (151.1, 116.8)
- added C8: 100n, Capacitor_SMD:C_1206_3216Metric_Pad1.42x1.75mm_HandSolder, F.Cu at (162.6, 71.1)
- added J4: ESP_PROG_JTAG, Connector_PinHeader_1.27mm:PinHeader_2x05_P1.27mm_Vertical, F.Cu at (137.2, 92.7)
- added J5: Prog, Connector_PinHeader_2.54mm:PinHeader_1x05_P2.54mm_Vertical, F.Cu at (161.9, 66.0)
- added J6: ext_Measure, Connector_Phoenix_MSTB:PhoenixContact_MSTBVA_2,5_4-G-5,08_1x04_P5.08mm_Vertical, F.Cu at (108.7, 94.5)
- added J7: Measurement-Selector, Connector_PinHeader_2.54mm:PinHeader_1x03_P2.54mm_Vertical, F.Cu at (115.8, 119.4)
- added J8: OLED_128x64, Connector_PinHeader_2.54mm:PinHeader_1x04_P2.54mm_Vertical, F.Cu at (173.7, 80.5)
- added Q1: UMH3N, lib_fp:SOT65P230X110-6N, F.Cu at (163.1, 61.0)
- added Q2: Si2302DS_NMOS, Package_TO_SOT_SMD:TSOT-23_HandSoldering, F.Cu at (117.3, 91.9)
- added Q3: Si2301DS_PMOS, Package_TO_SOT_SMD:TSOT-23_HandSoldering, F.Cu at (117.6, 86.6)
- added Q4: Si2302DS_NMOS, Package_TO_SOT_SMD:TSOT-23_HandSoldering, F.Cu at (165.6, 76.2)
- added Q5: Si2301DS_PMOS, Package_TO_SOT_SMD:TSOT-23_HandSoldering, F.Cu at (171.4, 71.1)
- added Q6: Si2302DS_NMOS, Package_TO_SOT_SMD:TSOT-23_HandSoldering, F.Cu at (172.2, 76.2)
- added R10: 10k, Resistor_SMD:R_1206_3216Metric_Pad1.42x1.75mm_HandSolder, F.Cu at (165.1, 71.1)
- added R11: 10k, Resistor_SMD:R_1206_3216Metric_Pad1.42x1.75mm_HandSolder, F.Cu at (170.7, 81.3)
- added R12: 100k, Resistor_SMD:R_1206_3216Metric_Pad1.42x1.75mm_HandSolder, F.Cu at (174.8, 70.9)
- added R13: 10k, Resistor_SMD:R_1206_3216Metric_Pad1.42x1.75mm_HandSolder, F.Cu at (168.1, 71.1)
- added R2: 10k, Resistor_SMD:R_1206_3216Metric_Pad1.42x1.75mm_HandSolder, F.Cu at (152.7, 89.7)
- added R3: 10k, Resistor_SMD:R_1206_3216Metric_Pad1.42x1.75mm_HandSolder, F.Cu at (121.9, 87.4)
- added R4: 10k, Resistor_SMD:R_1206_3216Metric_Pad1.42x1.75mm_HandSolder, F.Cu at (121.9, 92.5)
- added R5: optional, Resistor_SMD:R_1206_3216Metric_Pad1.42x1.75mm_HandSolder, F.Cu at (115.3, 101.6)
- added R6: optional, Resistor_SMD:R_1206_3216Metric_Pad1.42x1.75mm_HandSolder, F.Cu at (115.3, 96.6)
- added R7: 100k, Resistor_SMD:R_1206_3216Metric_Pad1.42x1.75mm_HandSolder, F.Cu at (117.9, 96.6)
- added R8: 100k, Resistor_SMD:R_1206_3216Metric_Pad1.42x1.75mm_HandSolder, F.Cu at (112.8, 86.6)
- added R9: 10k, Resistor_SMD:R_1206_3216Metric_Pad1.42x1.75mm_HandSolder, F.Cu at (170.7, 87.9)
- added TP1: TP_U_BATT, Connector_PinHeader_2.54mm:PinHeader_1x01_P2.54mm_Vertical, F.Cu at (126.5, 88.1)
- added TP2: TP_U_EXT, Connector_PinHeader_2.54mm:PinHeader_1x01_P2.54mm_Vertical, F.Cu at (126.5, 92.2)
- added TP3: VCC_2, Connector_PinHeader_2.54mm:PinHeader_1x01_P2.54mm_Vertical, F.Cu at (167.6, 86.4)
- BT1: footprint Connector_Phoenix_MSTB:PhoenixContact_MSTBA_2,5_2-G-5,08_1x02_P5.08mm_Horizontal -> Connector_Phoenix_MSTB:PhoenixContact_MSTBVA_2,5_2-G-5,08_1x02_P5.08mm_Vertical
- J3: footprint Connector_PinHeader_2.54mm:PinHeader_1x03_P2.54mm_Vertical -> Connector_PinHeader_2.54mm:PinHeader_1x05_P2.54mm_Vertical
- moved C1 17.6 mm to (117.1, 74.5)
- moved C2 17.6 mm to (123.0, 74.5)
- moved U1 17.6 mm to (119.4, 68.2)
- moved J3 15.5 mm to (115.3, 82.3), turned to 90 degrees
- moved BT1 6.75 mm to (109.2, 74.9), turned to 90 degrees
- moved J2 2.54 mm to (112.8, 61.0)
- moved J1 2.09 mm to (108.7, 85.0)
- moved U3 2.03 mm to (161.3, 110.6)
- moved AE1 2.03 mm to (173.7, 103.0)
- moved R1 1.15 mm to (128.5, 66.5), turned to 0 degrees
Connections:
- net Net-(BT1-Pad1) renamed /V-Batt
- net Net-(R1-Pad2) renamed /Reset
- C2 pad 1: Net-(C2-Pad1) -> +3V3
- C3 pad 1: +3V3 -> VCC
- C4 pad 1: +3V3 -> VCC
- J2 pad 2: +3V3 -> VCC
- J2 pad 3: Net-(C2-Pad1) -> +3V3
- R1 pad 1: +3V3 -> VCC
- U1 pad 3: Net-(C2-Pad1) -> +3V3
- U2 pad 10: Net-(U2-Pad10) -> /UBAT_ENABLE
- U2 pad 13: Net-(U2-Pad13) -> /TMS
- U2 pad 14: Net-(U2-Pad14) -> /TDI
- U2 pad 16: Net-(U2-Pad16) -> /TCK
- U2 pad 2: +3V3 -> VCC
- U2 pad 23: Net-(U2-Pad23) -> /TDO
- U2 pad 25: Net-(U2-Pad25) -> /Boot
- U2 pad 26: Net-(U2-Pad26) -> /U_EXT_ENABLE
- U2 pad 27: Net-(U2-Pad27) -> /POWER_ENABLE
- U2 pad 33: Net-(U2-Pad33) -> /SDA
- U2 pad 34: Net-(U2-Pad34) -> /RX
- U2 pad 35: Net-(U2-Pad35) -> /TX
- U2 pad 36: Net-(U2-Pad36) -> /SCL
- U2 pad 6: Net-(U2-Pad6) -> /UBAT_MEASURE
- U2 pad 7: Net-(U2-Pad7) -> /U_EXT_MEASURE
- U3 pad 13: +3V3 -> VCC
Routing:
- net VCC: track 0.00 -> 239.3 mm, vias 0 -> 9
- net /VCC_2: track 0.00 -> 107.8 mm, vias 0 -> 7
- net +3V3: track 98.1 -> 26.1 mm, vias 2 -> 0
- net /U_EXT_MEASURE: track 0.00 -> 52.3 mm, vias 0 -> 2
- net /U_EXT_ENABLE: track 0.00 -> 47.6 mm, vias 0 -> 3
- net /Reset: track 10.9 -> 50.1 mm
- net /SCL: track 0.00 -> 38.5 mm, vias 0 -> 5
- net /Boot: track 0.00 -> 36.7 mm, vias 0 -> 2
- net Net-(C2-Pad1): track 34.5 -> 0.00 mm, vias 2 -> 0
- net /POWER_ENABLE: track 0.00 -> 31.2 mm, vias 0 -> 2
- net /UBAT_MEASURE: track 0.00 -> 29.3 mm, vias 0 -> 1
- net /SDA: track 0.00 -> 27.8 mm, vias 0 -> 2
- net /UBAT_ENABLE: track 0.00 -> 26.5 mm
- net Net-(J6-Pad3): track 0.00 -> 26.1 mm
- net /SDA_2: track 0.00 -> 22.2 mm, vias 0 -> 2
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Other:
- net class Power added: clearance 0.2, trace_width 0.508, via_dia 1.016, via_drill 0.4

Commit message: .
Routing:
- net GND: track 33.0 -> 131.7 mm, vias 4 -> 14
- added copper zone on B.Cu, net GND
- added copper zone on F.Cu, net GND

Commit message: .
Parts:
- added REF**: KiCad-Logo2_6mm_SilkScreen, Symbol:KiCad-Logo2_6mm_SilkScreen, F.Cu at (140.0, 105.8)
- moved R9 1.17 mm to (169.9, 87.0)
- moved R11 0.92 mm to (169.9, 81.8)
- moved TP3 0.85 mm to (166.9, 86.0)
- moved R7 0.51 mm to (118.4, 96.6)
- moved R5 0.51 mm to (115.8, 101.6)
- moved R6 0.51 mm to (115.8, 96.6)
Routing:
- net Net-(J6-Pad3): track 26.1 -> 24.6 mm
- net /SDA_2: track 22.2 -> 21.0 mm
- net /U_EXT_ENABLE: track 47.6 -> 46.9 mm
- net /VCC_2: track 107.8 -> 108.4 mm
- net Net-(J6-Pad1): track 10.1 -> 10.6 mm
Other:
- board text added: "3.3V from USB"
- board text added: "DTR"
- board text added: "DUT"
- board text added: "Esp32LoraBoard V1.0 Viktor Rees"
- board text added: "R _low"
- board text added: "RTS"
- board text added: "RX"
- board text added: "R_high"
- board text added: "SCL"
- board text added: "SDA"
- board text added: "TX"
- board text added: "V-Batt"
- board text added: "VCC"
- board text added: "VCC_2"
- board text added: "ext.Volt."
- board text added: "external Voltage"
- board text removed: "3.3V"
- board text removed: "Bat"
- board text removed: "from Batttery"
- board text removed: "from USB"
